File: project1/OLED_driver.kicad_sch (KiCad schematic)
At the start: 16 parts, among them U41 REF5020IDGK, U42 OPA277UA, U43 MCP45HV31-ST

Commit message: update
Parts:
- R20: value 1K -> 750
Changed lines of the file:
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@@
     (pin "2")
     (instances
-      (project "demo_LMP7721"
+      (project "project1"
         (path "/17826947-3d7e-4fb5-aaf8-088579fef2d0/b4b10c2d-f2ab-4c1c-9ed1-34a3f61ff1d8"
           (reference "C81") (unit 1)
@@
     (pin "8")
     (instances
-      (project "demo_LMP7721"
+      (project "project1"
         (path "/17826947-3d7e-4fb5-aaf8-088579fef2d0/b4b10c2d-f2ab-4c1c-9ed1-34a3f61ff1d8"
           (reference "U41") (unit 1)
@@
     (pin "2")
     (instances
-      (project "demo_LMP7721"
+      (project "project1"
         (path "/17826947-3d7e-4fb5-aaf8-088579fef2d0/b4b10c2d-f2ab-4c1c-9ed1-34a3f61ff1d8"
           (reference "C79") (unit 1)
@@
     (pin "2")
     (instances
-      (project "demo_LMP7721"
+      (project "project1"
         (path "/17826947-3d7e-4fb5-aaf8-088579fef2d0/b4b10c2d-f2ab-4c1c-9ed1-34a3f61ff1d8"
           (reference "C80") (unit 1)
@@
     (pin "2")
     (instances
-      (project "demo_LMP7721"
+      (project "project1"
         (path "/17826947-3d7e-4fb5-aaf8-088579fef2d0/b4b10c2d-f2ab-4c1c-9ed1-34a3f61ff1d8"
           (reference "C82") (unit 1)
@@
     (pin "2")
     (instances
-      (project "demo_LMP7721"
+      (project "project1"
         (path "/17826947-3d7e-4fb5-aaf8-088579fef2d0/b4b10c2d-f2ab-4c1c-9ed1-34a3f61ff1d8"
           (reference "C95") (unit 1)
@@
       (effects (font (size 1.27 1.27)) (justify left))
     )
-    (property "Value" "1K" (at 172.72 132.08 90)
+    (property "Value" "750" (at 172.72 132.08 90)
       (effects (font (size 1.27 1.27)) (justify left))
     )
@@
     (pin "2")
     (instances
-      (project "demo_LMP7721"
+      (project "project1"
         (path "/17826947-3d7e-4fb5-aaf8-088579fef2d0/b4b10c2d-f2ab-4c1c-9ed1-34a3f61ff1d8"
           (reference "R20") (unit 1)
@@
     (pin "2")
     (instances
-      (project "demo_LMP7721"
+      (project "project1"
         (path "/17826947-3d7e-4fb5-aaf8-088579fef2d0/b4b10c2d-f2ab-4c1c-9ed1-34a3f61ff1d8"
           (reference "C137") (unit 1)
@@
     (pin "2")
     (instances
-      (project "demo_LMP7721"
+      (project "project1"
         (path "/17826947-3d7e-4fb5-aaf8-088579fef2d0/b4b10c2d-f2ab-4c1c-9ed1-34a3f61ff1d8"
           (reference "C83") (unit 1)
@@
     (pin "2")
     (instances
-      (project "demo_LMP7721"
+      (project "project1"
         (path "/17826947-3d7e-4fb5-aaf8-088579fef2d0/b4b10c2d-f2ab-4c1c-9ed1-34a3f61ff1d8"
           (reference "C130") (unit 1)
@@
     )
     (instances
-      (project "demo_LMP7721"
+      (project "project1"
         (path "/17826947-3d7e-4fb5-aaf8-088579fef2d0/b4b10c2d-f2ab-4c1c-9ed1-34a3f61ff1d8"
           (reference "U54") (unit 1)
@@
     (pin "2")
     (instances
-      (project "demo_LMP7721"
+      (project "project1"
         (path "/17826947-3d7e-4fb5-aaf8-088579fef2d0/b4b10c2d-f2ab-4c1c-9ed1-34a3f61ff1d8"
           (reference "C123") (unit 1)
@@
     (pin "9")
     (instances
-      (project "demo_LMP7721"
+      (project "project1"
         (path "/17826947-3d7e-4fb5-aaf8-088579fef2d0/b4b10c2d-f2ab-4c1c-9ed1-34a3f61ff1d8"
           (reference "U43") (unit 1)
@@
     (pin "2")
     (instances
-      (project "demo_LMP7721"
+      (project "project1"
         (path "/17826947-3d7e-4fb5-aaf8-088579fef2d0/b4b10c2d-f2ab-4c1c-9ed1-34a3f61ff1d8"
           (reference "R63") (unit 1)
@@
     (pin "2")
     (instances
-      (project "demo_LMP7721"
+      (project "project1"
         (path "/17826947-3d7e-4fb5-aaf8-088579fef2d0/b4b10c2d-f2ab-4c1c-9ed1-34a3f61ff1d8"
           (reference "R56") (unit 1)
@@
     (pin "8")
     (instances
-      (project "demo_LMP7721"
+      (project "project1"
         (path "/17826947-3d7e-4fb5-aaf8-088579fef2d0/b4b10c2d-f2ab-4c1c-9ed1-34a3f61ff1d8"
           (reference "U42") (unit 1)
