File: project1/amp.kicad_sch (KiCad schematic)
At the start: 17 parts, among them U10 REF102CU, U11 OPA277UA, U12 LMP7721MA

Commit message: update
Parts:
- R1: value 500K -> 510K
Changed lines of the file:
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@@
     (pin "8")
     (instances
-      (project "demo_LMP7721"
+      (project "project1"
         (path "/17826947-3d7e-4fb5-aaf8-088579fef2d0/f4a29f39-8e0c-4f92-96f5-fa4790ce3a68"
           (reference "U10") (unit 1)
@@
     (pin "2")
     (instances
-      (project "demo_LMP7721"
+      (project "project1"
         (path "/17826947-3d7e-4fb5-aaf8-088579fef2d0/f4a29f39-8e0c-4f92-96f5-fa4790ce3a68"
           (reference "C49") (unit 1)
@@
     (pin "8")
     (instances
-      (project "demo_LMP7721"
+      (project "project1"
         (path "/17826947-3d7e-4fb5-aaf8-088579fef2d0/f4a29f39-8e0c-4f92-96f5-fa4790ce3a68"
           (reference "U12") (unit 1)
@@
       (effects (font (size 1.27 1.27)) (justify right))
     )
-    (property "Value" "500K" (at 158.75 80.01 0)
+    (property "Value" "510K" (at 158.75 80.01 0)
       (effects (font (size 1.27 1.27)) (justify right))
     )
@@
     (pin "2")
     (instances
-      (project "demo_LMP7721"
+      (project "project1"
         (path "/17826947-3d7e-4fb5-aaf8-088579fef2d0/f4a29f39-8e0c-4f92-96f5-fa4790ce3a68"
           (reference "R1") (unit 1)
@@
     )
     (instances
-      (project "demo_LMP7721"
+      (project "project1"
         (path "/17826947-3d7e-4fb5-aaf8-088579fef2d0/f4a29f39-8e0c-4f92-96f5-fa4790ce3a68"
           (reference "U61") (unit 1)
@@
     (pin "2")
     (instances
-      (project "demo_LMP7721"
+      (project "project1"
         (path "/17826947-3d7e-4fb5-aaf8-088579fef2d0/f4a29f39-8e0c-4f92-96f5-fa4790ce3a68"
           (reference "C2") (unit 1)
@@
     (pin "8")
     (instances
-      (project "demo_LMP7721"
+      (project "project1"
         (path "/17826947-3d7e-4fb5-aaf8-088579fef2d0/f4a29f39-8e0c-4f92-96f5-fa4790ce3a68"
           (reference "U11") (unit 1)
@@
     (pin "2")
     (instances
-      (project "demo_LMP7721"
+      (project "project1"
         (path "/17826947-3d7e-4fb5-aaf8-088579fef2d0/f4a29f39-8e0c-4f92-96f5-fa4790ce3a68"
           (reference "C41") (unit 1)
@@
     (pin "2")
     (instances
-      (project "demo_LMP7721"
+      (project "project1"
         (path "/17826947-3d7e-4fb5-aaf8-088579fef2d0/f4a29f39-8e0c-4f92-96f5-fa4790ce3a68"
           (reference "R9") (unit 1)
@@
     (pin "2")
     (instances
-      (project "demo_LMP7721"
+      (project "project1"
         (path "/17826947-3d7e-4fb5-aaf8-088579fef2d0/f4a29f39-8e0c-4f92-96f5-fa4790ce3a68"
           (reference "C16") (unit 1)
@@
     (pin "2")
     (instances
-      (project "demo_LMP7721"
+      (project "project1"
         (path "/17826947-3d7e-4fb5-aaf8-088579fef2d0/f4a29f39-8e0c-4f92-96f5-fa4790ce3a68"
           (reference "R46") (unit 1)
@@
     (pin "2")
     (instances
-      (project "demo_LMP7721"
+      (project "project1"
         (path "/17826947-3d7e-4fb5-aaf8-088579fef2d0/f4a29f39-8e0c-4f92-96f5-fa4790ce3a68"
           (reference "C17") (unit 1)
@@
     (pin "2")
     (instances
-      (project "demo_LMP7721"
+      (project "project1"
         (path "/17826947-3d7e-4fb5-aaf8-088579fef2d0/f4a29f39-8e0c-4f92-96f5-fa4790ce3a68"
           (reference "C20") (unit 1)
@@
     (pin "2")
     (instances
-      (project "demo_LMP7721"
+      (project "project1"
         (path "/17826947-3d7e-4fb5-aaf8-088579fef2d0/f4a29f39-8e0c-4f92-96f5-fa4790ce3a68"
           (reference "R7") (unit 1)
@@
     (pin "2")
     (instances
-      (project "demo_LMP7721"
+      (project "project1"
         (path "/17826947-3d7e-4fb5-aaf8-088579fef2d0/f4a29f39-8e0c-4f92-96f5-fa4790ce3a68"
           (reference "R10") (unit 1)
@@
     (pin "2")
     (instances
-      (project "demo_LMP7721"
+      (project "project1"
         (path "/17826947-3d7e-4fb5-aaf8-088579fef2d0/f4a29f39-8e0c-4f92-96f5-fa4790ce3a68"
           (reference "C18") (unit 1)
@@
     (pin "2")
     (instances
-      (project "demo_LMP7721"
+      (project "project1"
         (path "/17826947-3d7e-4fb5-aaf8-088579fef2d0/f4a29f39-8e0c-4f92-96f5-fa4790ce3a68"
           (reference "C1") (unit 1)
